Commit message: Adjustments for day1 presentation

File: src/dynoturtle/dynoturtle_description/urdf/dynoturtle.xacro (robot description, xacro)
@@ -46,11 +46,4 @@
   <!-- Front bumper link -->
   <link name="${turtle_namespace}_front_bumper_link">
-    <visual>
-      <geometry>
-        <cylinder radius="${bumper_radius}" length="${bumper_height}"/>
-      </geometry>
-      <origin xyz="0 0 ${bumper_height/2}" rpy="0 0 0"/>
-      <material name="bumper_green"/>
-    </visual>
     <collision>
       <geometry>
