Commit message: Update from gazebo classic to harmonic

File: src/dynobot/dynobot_description/urdf/accessories/gazebo_control.xacro (robot description, xacro)
@@ -12,25 +12,25 @@
     </gazebo>
     <gazebo>
-        <plugin name="diff_drive" filename="libgazebo_ros_diff_drive.so">
+        <plugin name="gz::sim::systems::DiffDrive" filename="gz-sim-diff-drive-system">
             <!-- Wheel Information -->
             <left_joint>left_wheel_joint</left_joint>
             <right_joint>right_wheel_joint</right_joint>
             <wheel_separation>${dynobot_radius * 2}</wheel_separation>
-            <wheel_diameter>0.059*2</wheel_diameter>
-            <!-- Limits -->
-            <max_wheel_torque>200</max_wheel_torque>
-            <max_wheel_acceleration>5.0</max_wheel_acceleration>
+            <wheel_radius>0.059</wheel_radius>
+            <!-- Inputs -->
+            <topic>cmd_vel</topic>
             <!-- Outputs -->
-            <odometry_frame>odom</odometry_frame>
-            <robot_base_frame>base_link</robot_base_frame>
-            <publish_odom>true</publish_odom>
-            <publish_odom_tf>true</publish_odom_tf>
-            <publish_wheel_tf>true</publish_wheel_tf>
+            <frame_id>odom</frame_id>
+            <child_frame_id>base_link</child_frame_id>
+            <odom_topic>odom</odom_topic>
+            <odom_publisher_frequency>30</odom_publisher_frequency>
+            <tf_topic>/tf</tf_topic>
         </plugin>
-    </gazebo>
-        <plugin name="gazebo_ros_joint_state_publisher" filename="libgazebo_ros_joint_state_publisher.so">
-            <update_rate>20.0</update_rate>
+        <plugin filename="gz-sim-joint-state-publisher-system"
+            name="gz::sim::systems::JointStatePublisher">
+            <topic>joint_states</topic>
             <joint_name>left_wheel_joint</joint_name>
             <joint_name>right_wheel_joint</joint_name>
         </plugin>
+    </gazebo>
 </robot>

File: src/dynobot/dynobot_description/urdf/accessories/lidar.xacro (robot description, xacro)
@@ -1,7 +1,9 @@
 <?xml version="1.0"?>
 <robot xmlns:xacro="http://ros.org/wiki/xacro">
-  <xacro:macro name="lidar" params="frame topic parent_link min_angle max_angle min_range:=0.0 max_range:=100.0 *origin">
+  <xacro:macro name="lidar"
+    params="frame topic parent_link min_angle max_angle min_range:=0.0 max_range:=100.0 *origin">
     <!-- actual sample size = 2000 -->
-    <xacro:macro name="lslidar" params="frame:=laser_link topic:=scan sample_size:=720 update_rate:=10
+    <xacro:macro name="lslidar"
+      params="frame:=laser_link topic:=scan sample_size:=720 update_rate:=10
              min_range:=0.0 max_range:=100.0 robot_namespace:=/">
       <link name="${frame}_link">
@@ -16,9 +18,9 @@
       <gazebo reference="${frame}_link">
         <turnGravityOff>false</turnGravityOff>
-        <sensor type="ray" name="${frame}_link">
+        <sensor type="gpu_lidar" name="laser">
           <pose>0 0 0 0 0 0</pose>
           <visualize>false</visualize>
           <update_rate>${update_rate}</update_rate>
-          <ray>
+          <lidar>
             <scan>
               <horizontal>
@@ -39,8 +41,8 @@
               <stddev>0.001</stddev>
             </noise>
-          </ray>
-          <plugin name="gazebo_ros_${frame}"
-          filename="libgazebo_ros_ray_sensor.so">
-            <ros>
+          </lidar>
+          <topic>${topic}</topic>
+          <gz_frame_id>${frame}_link</gz_frame_id>
+          <!-- <ros>
               <remapping>~/out:=${topic}</remapping>
               <qos>
@@ -55,10 +57,10 @@
             <frame_name>${frame}_link</frame_name>
             <robot_namespace>${robot_namespace}</robot_namespace>
-            <output_type>sensor_msgs/LaserScan</output_type>
-          </plugin>
+            <output_type>sensor_msgs/LaserScan</output_type> -->
         </sensor>
       </gazebo>
     </xacro:macro>
-    <xacro:lslidar frame="${frame}" topic="${topic}" min_range="${min_range}" max_range="${max_range}"/>
+    <xacro:lslidar frame="${frame}" topic="${topic}" min_range="${min_range}"
+      max_range="${max_range}" />
     <joint name="${frame}_mount_joint" type="fixed">
       <xacro:insert_block name="origin" />

File: src/dynobot/dynobot_description/urdf/dynobot.xacro (robot description, xacro)
@@ -6,5 +6,5 @@
   <xacro:property name="turtle_radius" value="0.3" />
   <xacro:property name="turtle_height" value="0.2" />
-  <xacro:property name="turtle_mass" value="5.0" />
+  <xacro:property name="turtle_mass" value="10" />
   <xacro:property name="use_lidar" value="true" />
   <xacro:property name="lidar_min_range" value="0.06" />
@@ -22,5 +22,5 @@
     <parent link="base_link" />
     <child link="chassis_link" />
-    <origin xyz="0 0 0" rpy="0 0 0" />
+    <origin xyz="0 0 ${turtle_height/2}" rpy="0 0 0" />
   </joint>
   <!-- Base link (simple cylinder turtle body) -->
@@ -31,5 +31,5 @@
       </geometry>
       <material name="dyno_green" />
-      <origin xyz="0 0 ${turtle_height/2}" rpy="0 0 0" />
+      <origin xyz="0 0 0" rpy="0 0 0" />
     </visual>
     <collision>
@@ -37,5 +37,5 @@
         <cylinder radius="${turtle_radius}" length="${turtle_height}" />
       </geometry>
-      <origin xyz="0 0 ${turtle_height/2}" rpy="0 0 0" />
+      <origin xyz="0 0 0" rpy="0 0 0" />
     </collision>
     <xacro:inertial_cylinder mass="${turtle_mass}" radius="${turtle_radius}"
@@ -46,5 +46,5 @@
   <!-- Caster Wheel -->
   <joint name="caster_wheel_joint" type="fixed">
-    <parent link="chassis_link" />
+    <parent link="base_link" />
     <child link="caster_wheel" />
     <origin xyz="${turtle_radius*3/4} 0 0" rpy="0 0 0" />
@@ -64,5 +64,5 @@
       <origin xyz="0 0 0" rpy="0 0 0" />
     </collision>
-    <xacro:inertial_sphere mass="1" radius="0.059">
+    <xacro:inertial_sphere mass="0.1" radius="0.059">
       <origin xyz="0 0 0" rpy="0 0 0" />
     </xacro:inertial_sphere>
@@ -78,6 +78,6 @@
   <xacro:if value="${use_lidar}">
     <xacro:lidar frame="laser" topic="/scan" parent_link="chassis_link" min_angle="${-PI}"
-                max_angle="${PI}" min_range="${lidar_min_range}" max_range="${lidar_max_range}">
-      <origin xyz="0 0 ${turtle_height}" rpy="0 0 0" />
+      max_angle="${PI}" min_range="${lidar_min_range}" max_range="${lidar_max_range}">
+      <origin xyz="0 0 ${turtle_height/2}" rpy="0 0 0" />
     </xacro:lidar>
   </xacro:if>
